Commit message: Aufgabe_1

File: packages/src/auna_gazebo/models/race_car/model.urdf (robot description, URDF)
Before this commit: robot sam_bot, 6 links, 5 joints
Links:
- added link $(arg namespace)marker_1, mass 0.01; collision sphere radius=0.05; visual sphere radius=0.05
- added link $(arg namespace)marker_2, mass 0.01; collision sphere radius=0.05; visual sphere radius=0.05
- added link $(arg namespace)marker_3, mass 0.01; collision sphere radius=0.05; visual sphere radius=0.05
Joints:
- added joint marker_1_joint: type fixed, parent $(arg namespace)chassis, child $(arg namespace)marker_1, origin xyz=0.2 0.0 0.2 rpy=0 0 0
- added joint marker_2_joint: type fixed, parent $(arg namespace)chassis, child $(arg namespace)marker_2, origin xyz=-0.1 0.1 0.2 rpy=0 0 0
- added joint marker_3_joint: type fixed, parent $(arg namespace)chassis, child $(arg namespace)marker_3, origin xyz=-0.1 -0.1 0.2 rpy=0 0 0

Commit message: hungarian_going

File: packages/src/auna_gazebo/models/race_car/model.urdf (robot description, URDF)
Before this commit: robot sam_bot, 9 links, 8 joints
Links:
- added link $(arg namespace)marker_4, mass 0.01; collision sphere radius=0.01; visual sphere radius=0.01
- link $(arg namespace)marker_1: geometry collision sphere radius=0.01; visual sphere radius=0.01
- link $(arg namespace)marker_2: geometry collision sphere radius=0.01; visual sphere radius=0.01
- link $(arg namespace)marker_3: geometry collision sphere radius=0.01; visual sphere radius=0.01
Joints:
- added joint marker_4_joint: type fixed, parent $(arg namespace)chassis, child $(arg namespace)marker_4, origin xyz=0.22 -0.07 0.2 rpy=0 0 0
- joint marker_1_joint: origin xyz=0.2 0.0 0.2 rpy=0 0 0 -> xyz=0.1 0.0 0.2 rpy=0 0 0
- joint marker_2_joint: origin xyz=-0.1 0.1 0.2 rpy=0 0 0 -> xyz=-0.12 0.025 0.2 rpy=0 0 0
- joint marker_3_joint: origin xyz=-0.1 -0.1 0.2 rpy=0 0 0 -> xyz=-0.12 -0.025 0.2 rpy=0 0 0

Commit message: ekf_problem

File: packages/src/auna_gazebo/models/race_car/model.urdf (robot description, URDF)
Before this commit: robot sam_bot, 10 links, 9 joints
Links:
- removed link $(arg namespace)base_link
- removed link $(arg namespace)camera
- removed link $(arg namespace)chassis
- removed link $(arg namespace)imu_link
- removed link $(arg namespace)laser
- removed link $(arg namespace)marker_1
- removed link $(arg namespace)marker_2
- removed link $(arg namespace)marker_3
- removed link $(arg namespace)marker_4
- removed link $(arg namespace)steering_wheel
- added link base_link
- added link camera, mass ${cameraMass}; collision box size=${cameraSizeL} ${cameraSizeH} ${cameraSizeB}; visual mesh filename=file:///$(find auna_gazebo)/models/race_car/meshes/ZED.dae
- added link chassis, mass ${bodyMass}; collision box size=${bodySizeL} ${bodySizeB} ${bodySizeH}; visual mesh filename=file:///$(find auna_gazebo)/models/race_car/meshes/car.dae
- added link imu_link
- added link laser, mass ${hokuyoMass}; collision box size=${hokuyoSize} ${hokuyoSize} ${hokuyoSize}; visual mesh filename=file:///$(find auna_gazebo)/models/race_car/meshes/hokuyo.d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
- added link marker_1, mass 0.01; collision sphere radius=0.01; visual sphere radius=0.01
- added link marker_2, mass 0.01; collision sphere radius=0.01; visual sphere radius=0.01
- added link marker_3, mass 0.01; collision sphere radius=0.01; visual sphere radius=0.01
- added link marker_4, mass 0.01; collision sphere radius=0.01; visual sphere radius=0.01
- added link steering_wheel, mass 0.1; collision box size=0.01 0.01 0.01; visual box size=0.01 0.01 0.01
Joints:
- joint base_link_joint: child $(arg namespace)chassis -> chassis; parent $(arg namespace)base_link -> base_link
- joint camera_joint: child $(arg namespace)camera -> camera; parent $(arg namespace)chassis -> chassis
- joint imu_joint: child $(arg namespace)imu_link -> imu_link; parent $(arg namespace)chassis -> chassis
- joint laser_joint: child $(arg namespace)laser -> laser; parent $(arg namespace)chassis -> chassis
- joint marker_1_joint: child $(arg namespace)marker_1 -> marker_1; parent $(arg namespace)chassis -> chassis
- joint marker_2_joint: child $(arg namespace)marker_2 -> marker_2; parent $(arg namespace)chassis -> chassis
- joint marker_3_joint: child $(arg namespace)marker_3 -> marker_3; parent $(arg namespace)chassis -> chassis
- joint marker_4_joint: child $(arg namespace)marker_4 -> marker_4; parent $(arg namespace)chassis -> chassis
- joint steering_wheel_joint: child $(arg namespace)steering_wheel -> steering_wheel; parent $(arg namespace)chassis -> chassis

Commit message: updated working config

File: packages/src/auna_gazebo/models/race_car/model.urdf (robot description, URDF)
Before this commit: robot sam_bot, 10 links, 9 joints
Links:
- added link gps_link, mass ${gpsMass}; collision box size=${gpsSizeL} ${gpsSizeB} ${gpsSizeH}; visual box size=${gpsSizeL} ${gpsSizeB} ${gpsSizeH}
- link imu_link: mass None -> 0.01
Joints:
- added joint gps_joint: type fixed, parent chassis, child gps_link, origin xyz=-0.1 0 0.15 rpy=0 0 0

Commit message: basic code completed

File: packages/src/auna_gazebo/models/race_car/model.urdf (robot description, URDF)
Before this commit: robot sam_bot, 11 links, 10 joints
Links:
- link marker_1: mass 0.01 -> 0.0
- link marker_2: mass 0.01 -> 0.0
- link marker_3: mass 0.01 -> 0.0
- link marker_4: mass 0.01 -> 0.0
